Commit message: Refactor Icebot robot model: remove old test notebook, add new advances notebook, and update URDF with tool joint

File: docs/robot/icebot.urdf (robot description, URDF)
Before this commit: robot icebot, 5 links, 4 joints
Links:
- added link tool0
Joints:
- added joint tcp_joint: type fixed, parent end_effector, child tool0, origin xyz=0 0 -0.12 rpy=0 0 0
