Commit message: FIN

File: docs/execution/robot/icebot.urdf (robot description, URDF)
Before this commit: robot icebot, 6 links, 5 joints
Joints:
- joint axis_0: origin xyz=0 0 0.1 rpy=0 0 0 -> xyz=0 0 0.1 rpy=0 0 0.3491
- joint axis_1: limit lower=0.0 upper=2.0944 effort=10.0 velocity=1.0 -> lower=-1.5708 upper=1.5708 effort=10.0 velocity=1.0

Commit message: Refactor code structure for improved readability and maintainability

File: docs/execution/robot/icebot.urdf (robot description, URDF)
Before this commit: robot icebot, 6 links, 5 joints
Joints:
- joint axis_1: limit lower=-1.5708 upper=1.5708 effort=10.0 velocity=1.0 -> lower=-2.0944 upper=2.0944 effort=10.0 velocity=1.0
